Commit message: Session3 Completed

File: session3/diff_robot_description/urdf/diff_robot.urdf (robot description, URDF)
Before this commit: robot diff_robot, 5 links, 4 joints
Links:
- link base_link: mass None -> 5; geometry collision box size=0.6 0.4 0.2; visual box size=0.6 0.4 0.2
- link caster_wheel_link: mass None -> 0.5; geometry collision sphere radius=0.05; visual sphere radius=0.05
- link left_wheel_link: mass None -> 1; geometry collision cylinder length=0.05 radius=0.1; visual cylinder length=0.05 radius=0.1
- link right_wheel_link: mass None -> 1; geometry collision cylinder length=0.05 radius=0.1; visual cylinder length=0.05 radius=0.1

Commit message: Session4 part 2.1

File: session3/diff_robot_description/urdf/diff_robot.urdf (robot description, URDF)
Before this commit: robot diff_robot, 5 links, 4 joints
Links:
- added link imu_link, mass 0.5; collision box size=0.05 0.05 0.02; visual box size=0.05 0.05 0.02
- added link lidar_link, mass 0.5; collision cylinder length=0.05 radius=0.06; visual cylinder length=0.05 radius=0.06
Joints:
- added joint base_imu_joint: type fixed, parent base_link, child imu_link, origin xyz=0 0 0.01 rpy=0 0 0
- added joint base_lidar_joint: type fixed, parent base_link, child lidar_link, origin xyz=0 0 0.225 rpy=0 0 0
